File: hardware/kicad/pendulum_control_board.sch (KiCad schematic (older format))
At the start: 263 parts, among them IC1 STM32F411CEU6, IC2 LM358D, J1 DX07S024JJ2, Q1 BSS138, Q2 BSS138, Q3 BSS138, Q4 BSS138, Q5 2N7002, Q6 2N7002, Q7 2N7002, U1 FT231XS, U2 V_REG_317SMD, U3 V_REG_317SMD, U5 LTC6102DD, X1 5566-8, X2 5566-8, Y2 32.768kHz

Commit message: added schottkys to charging circuit
Parts:
- added D1, D17: MBR0520, Diodes_SMD:SOD-123, symbol MBR0520
Connections:
- net GND: now also D1.2 (A), D17.2 (A)
- net N$62: now also D1.1 (K)
- net N$65: now also D17.1 (K)

Commit message: added bom and updated board
Parts:
- removed D11, D12, D13, D14: 1N4148, ADAFRUIT_SOT23-R, symbol ADAFRUIT_DIODESOT23_REFLOW
- added D11, D12, D13, D14: 1N4148, Diodes_SMD:SOD-123, symbol 1N4148
- C36, C39, C42, C45: footprint SPARKFUN-CAPACITORS_0603 -> Capacitors_SMD:C_1206
- R105: value (none) -> 100K
- R43, R56: value (none) -> 5.6K
- R47, R65: value 185K -> 187K
- R49, R62: value (none) -> 1M
- R50, R63: value (none) -> 4.7K
- R51, R64: value (none) -> 1K
- R75: value (none) -> 4.7
- R78: value (none) -> 402K
- R79: value (none) -> 107K
- R81, R82, R86, R87: value (none) -> 1
- R83: value (none) -> 0
- R84: value (none) -> 2K
- R85: value (none) -> 115K
- R88: value (none) -> 0.01
- R99: footprint SPARKFUN-RESISTORS_0603 -> Resistors_SMD:R_1206
Connections:
- net N$45: now also D13.1 (K)
- net N$47: now also D11.1 (K)
- net V_DRIVER_X: now also D12.2 (A)
- net V_DRIVER_Y: now also D14.2 (A)
- net N$46: no longer names the net of R54.2
- net N$46: now also D13.2 (A), D14.1 (K)
- net N$48: no longer names the net of R41.2
- net N$48: now also D11.2 (A), D12.1 (K)
Other:
- note added: "NOTE: 80 Ohm resistor sets FREQ to 1200 kHz, 187 KOhm sets V_DRIVER close to 24 V"
- note removed: "NOTE: 80 Ohm resistor sets FREQ to 1200 kHz, 185 KOhm sets V_DRIVER to 24 V"
